File: input/routed/right.kicad_pcb (KiCad board)
At the start: 2 copper layers, 90 x 71 mm, 44 parts, among them T2 Flactyl 4.0 (left)

Commit message: All is cool!
Parts:
- moved D7 8.88 mm to (32.4, -45.6)
- moved D10 8.88 mm to (14.4, -39.6)
- moved D11 8.88 mm to (14.4, -22.6)
- moved D1 8.88 mm to (75.6, -20.4)
- moved D2 8.88 mm to (75.6, -3.40)
- moved D3 8.88 mm to (75.6, 13.6)
- moved H6 1.00 mm to (9.00, -43.5)
Routing:
- net R0: track 0.00 -> 194.7 mm, vias 0 -> 6
- net GND: track 0.00 -> 156.9 mm, vias 0 -> 4
- net R2: track 0.00 -> 135.4 mm, vias 0 -> 4
- net R1: track 0.00 -> 128.8 mm, vias 0 -> 7
- net C0: track 35.1 -> 143.6 mm, vias 0 -> 1
- net RAW: track 0.00 -> 106.7 mm, vias 0 -> 1
- net R3: track 0.00 -> 101.5 mm, vias 0 -> 2
- net C1: track 35.1 -> 113.1 mm, vias 0 -> 3
- net P2: track 0.00 -> 73.7 mm, vias 0 -> 4
- net P3: track 0.00 -> 72.4 mm
- net C2: track 35.1 -> 88.9 mm, vias 0 -> 1
- net C6: track 0.00 -> 53.1 mm, vias 0 -> 2
- net C5: track 0.00 -> 52.7 mm, vias 0 -> 2
- net RST: track 0.00 -> 49.8 mm, vias 0 -> 1
- net C4: track 0.00 -> 44.6 mm, vias 0 -> 2
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Other:
- outline, holes or cut-outs redrawn

Commit message: Fix rounting right
Parts:
- moved H6 0.50 mm to (9.00, -44.0)
- turned J1 to 90 degrees
- turned JST1 to 90 degrees
Routing:
- net GND: track 156.9 -> 141.4 mm, vias 4 -> 5
- net C5: track 52.7 -> 62.7 mm
- net R0: track 194.7 -> 187.0 mm
- net R1: track 128.8 -> 123.9 mm, vias 7 -> 6
- net R2: track 135.4 -> 130.7 mm, vias 4 -> 5
- net C6: track 53.1 -> 57.7 mm, vias 2 -> 0
- net BSLI: track 23.5 -> 25.0 mm
