File: input/routed/right.kicad_pcb (KiCad board)
At the start: 2 copper layers, 90 x 71 mm, 44 parts, among them T1 Flactyl 4.0 (left)

Commit message: Fix
Parts:
- SS1: value (none) -> SW-TH_MSK12C02-HB-1
- T1: value Flactyl 4.0 (left) -> Flactyl 4.1 (left)
- turned SS1 to 180 degrees

Commit message: 4.1
Parts:
- moved H6 15.7 mm to (11.5, -28.5)
- moved D15 8.88 mm to (3.60, 2.60), turned to 0 degrees
- moved H5 8.50 mm to (9.00, -3.00)
- turned S15 to 0 degrees
Routing:
- net C6: track 57.7 -> 50.6 mm
- net C1: track 113.1 -> 117.1 mm
- net C4R2D: track 3.77 -> 0.00 mm
- net RAW: track 107.1 -> 103.5 mm, vias 1 -> 0
- net R2: track 130.7 -> 134.0 mm, vias 5 -> 6
- net P3: track 72.4 -> 75.4 mm, vias 0 -> 2
- net C4: track 44.6 -> 45.8 mm, vias 2 -> 1
- net P2: track 73.7 -> 74.4 mm
Other:
- outline, holes or cut-outs redrawn
