File: input/routed/right.kicad_pcb (KiCad board)
At the start: 2 copper layers, 90 x 71 mm, 44 parts, among them T1 Flactyl 4.1 (left)

Commit message: Update routed
Parts:
- removed H6: , MountingHole_2.2mm_M2
- T1: value Flactyl 4.1 (left) -> Flactyl 4.2 (right)
- moved D16 86.1 mm to (3.60, 2.60), turned to 0 degrees
- moved D1 72.8 mm to (3.60, -31.4)
- moved D2 72.8 mm to (3.60, -14.4)
- moved S1 72.8 mm to (0.00, -34.0)
- moved S2 72.8 mm to (0.00, -17.0)
- moved H1 60.1 mm to (11.5, -28.5)
- moved D3 57.6 mm to (76.0, -44.0), turned to 180 degrees
- moved H5 54.3 mm to (63.0, 2.50)
- moved S4 38.5 mm to (72.0, -6.00), turned to 0 degrees
- moved S5 38.5 mm to (72.0, 11.0), turned to 0 degrees
- moved S12 34.0 mm to (18.0, -37.0)
- moved S3 34.0 mm to (72.0, -23.0)
- moved S6 34.0 mm to (54.0, -40.0)
- moved S9 34.0 mm to (36.0, -43.0)
- moved D4 33.6 mm to (75.6, -20.4), turned to 0 degrees
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Connections:
- D1 pad 2: C0R0D -> C4_R0D
- D10 pad 2: C3R0D -> C2_R0D
- D11 pad 2: C3R1D -> C2_R1D
- D12 pad 2: C3R2D -> C2_R2D
- D13 pad 2: C4R0D -> C3_R0D
- D14 pad 2: C4R1D -> C3_R1D
- D15 pad 2: C4R2D -> C3_R2D
- D16 pad 1: R3 -> R2
- D16 pad 2: C0R3D -> C4_R2D
- D2 pad 2: C0R1D -> C4_R1D
- D3 pad 1: R2 -> R3
- D3 pad 2: C0R2D -> C0R3D
- D4 pad 2: C1R0D -> C0_R0D
- D5 pad 2: C1R1D -> C0_R1D
- D6 pad 2: C1R2D -> C0_R2D
- D7 pad 2: C2R0D -> C1_R0D
- D8 pad 2: C2R1D -> C1_R1D
- D9 pad 2: C2R2D -> C1_R2D
- S1 pad 1: C0R0D -> C4_R0D
- S1 pad 2: C0 -> C4
- S10 pad 1: C3R0D -> C2_R1D
- S10 pad 2: C3 -> C2
- S10 pad 3: C3R0D -> C2_R1D
- S10 pad 4: C3 -> C2
- S11 pad 1: C3R1D -> C2_R2D
- S11 pad 2: C3 -> C2
- S11 pad 3: C3R1D -> C2_R2D
- S11 pad 4: C3 -> C2
- S12 pad 1: C3R2D -> C3_R0D
- S12 pad 3: C3R2D -> C3_R0D
- S13 pad 1: C4R0D -> C3_R1D
- S13 pad 2: C4 -> C3
- S14 pad 1: C4R1D -> C3_R2D
- S14 pad 2: C4 -> C3
- S15 pad 1: C4R2D -> C4_R2D
- S15 pad 3: C4R2D -> C4_R2D
- S2 pad 1: C0R1D -> C4_R1D
- S2 pad 2: C0 -> C4
- S3 pad 1: C0R2D -> C0_R0D
- S3 pad 3: C0R2D -> C0_R0D
- S4 pad 1: C1R0D -> C0_R1D
- S4 pad 2: C1 -> C0
- S4 pad 3: C1R0D -> C0_R1D
- S4 pad 4: C1 -> C0
- S5 pad 1: C1R1D -> C0_R2D
- S5 pad 2: C1 -> C0
- S5 pad 3: C1R1D -> C0_R2D
- S5 pad 4: C1 -> C0
- S6 pad 1: C1R2D -> C1_R0D
- S6 pad 3: C1R2D -> C1_R0D
- S7 pad 1: C2R0D -> C1_R1D
- S7 pad 2: C2 -> C1
- S7 pad 3: C2R0D -> C1_R1D
- S7 pad 4: C2 -> C1
- S8 pad 1: C2R1D -> C1_R2D
- S8 pad 2: C2 -> C1
- S8 pad 3: C2R1D -> C1_R2D
- S8 pad 4: C2 -> C1
- S9 pad 1: C2R2D -> C2_R0D
- S9 pad 3: C2R2D -> C2_R0D
Routing:
- net C4_R1D: track 0.00 -> 9.80 mm
- net C4_R0D: track 0.00 -> 9.80 mm
- net C4R1D: track 9.80 -> 0.00 mm
- net C4R0D: track 9.80 -> 0.00 mm
- net C4_R2D: track 0.00 -> 7.89 mm, vias 0 -> 2
- net C4R2D: track 7.89 -> 0.00 mm, vias 2 -> 0
- net C2_R0D: track 0.00 -> 3.77 mm
- net C2R0D: track 3.77 -> 0.00 mm
- net C3_R0D: track 0.00 -> 3.77 mm
- net C3R0D: track 3.77 -> 0.00 mm
- net C2_R2D: track 0.00 -> 3.77 mm
- net C2R2D: track 3.77 -> 0.00 mm
- net C1_R0D: track 0.00 -> 3.77 mm
- net C1R0D: track 3.77 -> 0.00 mm
- net C3_R2D: track 0.00 -> 3.77 mm
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
Commit message: V5 pcbs
Parts:
- SS1: value SW-TH_MSK12C02-HB-1 -> SW-SMD_SS-3235D-03-L2.00; footprint easyeda:SW-TH_MSK12C02-HB-1 -> SW-SMD_SS-3235D-03-L2.00; moved to B.Cu
- T1: value Flactyl 4.2 (right) -> Flactyl 5.0 (right)
- moved SB1 44.6 mm to (58.5, -17.5), turned to 90 degrees
- moved SS1 23.9 mm to (51.5, -18.2)
- moved JC1 19.9 mm to (40.0, -20.5)
- moved JB1 16.0 mm to (58.0, -2.00)
- moved D3 7.00 mm to (76.0, -37.0)
- moved T1 3.16 mm to (35.5, -1.50)
Connections:
- net C0R3D renamed C0_R3D
Routing:
- net GND: track 141.4 -> 0.00 mm, vias 5 -> 0
- net RST: track 49.9 -> 86.9 mm, vias 1 -> 2
- net R0: track 187.0 -> 150.7 mm, vias 6 -> 7
- net R3: track 101.5 -> 124.0 mm, vias 2 -> 4
- net C0: track 143.6 -> 156.1 mm, vias 1 -> 3
- net C5: track 62.7 -> 52.5 mm
- net RAW: track 103.5 -> 93.5 mm, vias 0 -> 2
- net C6: track 50.6 -> 60.3 mm, vias 0 -> 2
- net C0_R3D: track 3.23 -> 11.6 mm
- net R2: track 134.0 -> 141.4 mm, vias 6 -> 8
- net C1: track 117.1 -> 112.1 mm, vias 3 -> 2
- net P3: track 75.4 -> 80.2 mm, vias 2 -> 3
- net C3: track 74.4 -> 69.8 mm, vias 1 -> 0
- net BSLI: track 25.0 -> 29.5 mm
- net C4_R2D: track 7.89 -> 3.77 mm, vias 2 -> 0
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Other:
- outline, holes or cut-outs redrawn

Commit message: Fix righnt
Routing:
- net C0: track 156.1 -> 157.7 mm
- net P2: track 71.7 -> 72.5 mm
- net RST: track 86.9 -> 87.6 mm

Commit message: PCB 5.1
Parts:
- T1: value Flactyl 5.0 (right) -> Flactyl 5.1 (right)
Routing:
- net C0: track 157.7 -> 160.9 mm
- net P2: track 72.5 -> 75.4 mm
- net RST: track 87.6 -> 88.7 mm
- net C1: track 112.5 -> 113.6 mm
