File: input/routed/thumb.kicad_pcb (KiCad board)
At the start: 2 copper layers, 36 x 51 mm, 18 parts, among them T1 Flactyl 4.2 (thumb), T2 x, T3 y

Commit message: PCB 5.1
Parts:
- T1: value Flactyl 4.2 (thumb) -> Flactyl 5.1 (thumb)
Routing:
- net R2: track 63.1 -> 69.6 mm
- net C6: track 56.7 -> 59.8 mm
- net C5: track 42.5 -> 45.1 mm
