File: input/schema/left.kicad_sch (KiCad schematic)
At the start: 35 parts, among them J1 Conn_01x05_Female, J2 Conn_01x02_Male, SW1 SW_DIP_x01, SW2 SW_DPDT_x2, U1 nice_nano

Commit message: Clean up build, soon will be jlcpcb
Parts:
- added D16: DIODE, Yan libraryo:D_SOD-523, symbol yan_Library:DIODE
- added SW3: RotaryEncoder_Switch, symbol Device:RotaryEncoder_Switch
Connections:
- net B-: now also SW3.C
- net Col0: now also SW3.S1
- net Row3: now reaches U1.10 (P0.11)
- net Row3: now also D16.1 (A)
- net Ro1: now reaches U1.5 (P0.17)
- net Ro1: now also SW3.A
- net Ro2: now reaches U1.6 (P0.20)
- net Ro2: now also SW3.B
- new net: D16.2 (K), SW3.S2
