File: input/schema/right.kicad_sch (KiCad schematic)
At the start: 35 parts, among them J1 Conn_01x05_Female, J2 Conn_01x02_Male, SW1 SW_DPDT_x2, U1 nice_nano

Commit message: Clean up build, soon will be jlcpcb
Parts:
- added D16: DIODE, Yan libraryo:D_SOD-523, symbol yan_Library:DIODE
- added SW2: RotaryEncoder_Switch, symbol Device:RotaryEncoder_Switch
Connections:
- net B-: now also SW2.C
- net Col0: now also SW2.S1
- net Row3: now reaches U1.10 (P0.11)
- net Row3: now also D16.1 (A)
- net Ro1: now reaches U1.5 (P0.17)
- net Ro1: now also SW2.A
- net Ro2: now reaches U1.6 (P0.20)
- net Ro2: now also SW2.B
- new net: D16.2 (K), SW2.S2
