File: 4.0/left/left.kicad_pcb (KiCad board)
At the start: 2 copper layers, 90 x 71 mm, 44 parts, among them T1 Flactyl 4.0 (left)

Commit message: Add 4.1
Parts:
- T1: moved to F.SilkS
Routing:
- net C0R0: track 0.00 -> 188.4 mm, vias 0 -> 1
- net R0: track 188.4 -> 3.77 mm, vias 1 -> 0
- net P3: track 183.5 -> 0.00 mm
- net C3R0D: track 3.77 -> 183.5 mm
- net P2: track 163.6 -> 0.00 mm
- net C0R1D: track 3.77 -> 164.4 mm, vias 0 -> 4
- net GND: track 138.6 -> 0.00 mm, vias 5 -> 0
- net C3R0: track 0.00 -> 138.6 mm, vias 0 -> 5
- net R2: track 122.7 -> 3.77 mm, vias 2 -> 0
- net C3: track 53.2 -> 163.6 mm
- net R3: track 109.4 -> 0.00 mm
- net C3R1D: track 3.77 -> 109.4 mm
- net C2: track 83.9 -> 3.77 mm, vias 1 -> 0
- net C1R0D: track 3.77 -> 83.9 mm, vias 0 -> 1
- net RAW: track 77.8 -> 0.00 mm, vias 2 -> 0
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Other:
- net class Default added: clearance 0.2, trace_width 0.25, via_dia 0.8, via_drill 0.4
