File: 4.0/right/right.kicad_pcb (KiCad board)
At the start: 2 copper layers, 90 x 71 mm, 44 parts, among them T1 Flactyl 4.0 (left)

Commit message: Add 4.1
Parts:
- T1: moved to F.SilkS
Routing:
- net C0R0: track 0.00 -> 187.0 mm, vias 0 -> 6
- net R0: track 187.0 -> 3.77 mm, vias 6 -> 0
- net GND: track 141.4 -> 0.00 mm, vias 5 -> 0
- net C3R0: track 0.00 -> 141.4 mm, vias 0 -> 5
- net R2: track 130.7 -> 3.77 mm, vias 5 -> 0
- net C0R1D: track 3.77 -> 123.9 mm, vias 0 -> 6
- net C1: track 113.1 -> 3.77 mm, vias 3 -> 0
- net C0R2D: track 3.77 -> 113.1 mm, vias 0 -> 3
- net RAW: track 107.1 -> 0.00 mm, vias 1 -> 0
- net C3R1: track 0.00 -> 107.1 mm, vias 0 -> 1
- net R3: track 101.5 -> 0.00 mm, vias 2 -> 0
- net C3R1D: track 3.77 -> 101.5 mm, vias 0 -> 2
- net C2: track 88.9 -> 3.77 mm, vias 1 -> 0
- net C1R0D: track 3.77 -> 88.9 mm, vias 0 -> 1
- net P2: track 73.7 -> 0.00 mm, vias 4 -> 0
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Other:
- net class Default added: clearance 0.2, trace_width 0.25, via_dia 0.8, via_drill 0.4
