File: 4.0/thumb/thumb.kicad_pcb (KiCad board)
At the start: 2 copper layers, 36 x 51 mm, 19 parts, among them T1 Flactyl 4.0 (thumb), T2 x, T3 y

Commit message: Add 4.1
Parts:
- T1, T2, T3: moved to F.SilkS
Routing:
- net R2: track 62.7 -> 3.77 mm
- net C6: track 57.9 -> 3.77 mm
- net C5R2D: track 3.77 -> 57.9 mm
- net C5R0: track 0.00 -> 43.2 mm
- net R0: track 43.2 -> 3.77 mm
- net R1: track 29.7 -> 62.7 mm
- net C5R1D: track 3.77 -> 29.7 mm
- net C6R0D: track 3.77 -> 0.00 mm
- net C5R2: track 0.00 -> 3.77 mm
- net C5R1: track 0.00 -> 3.77 mm
- net C6R2D: track 3.77 -> 0.00 mm
- net C6R1D: track 3.77 -> 0.00 mm
Other:
- net class Default added: clearance 0.2, trace_width 0.25, via_dia 0.8, via_drill 0.4
